File: Eagle/PowerWaechter.sch (EAGLE design)
At the start: 13 parts, among them U1 ESP32-DEVKITC-32D, X1 12V, X2 JST-XH-03-PIN-ROUND-PAD, X3 JST-XH-03-PIN-ROUND-PAD, X4 Versorgung, X5 230V | N | L

Commit message: v2.0.0 überführt
Parts:
- removed X1: 12V, con-wago-500:W237-102
- removed X2, X3: JST-XH-03-PIN-ROUND-PAD, Rembrandt Electronics - JST XH Connectors v1-0:JST-XH-03-PIN-ROUND-PAD
- removed X4: Versorgung, con-wago-500:W237-102
- removed X5: 230V | N | L, con-wago-500:W237-102
- added CON1, CON2: JST-XH-03, PowerGuard:JST-XH-03
- added CON3, CON4: (no value), PowerGuard:WAGO-500-2
- added LED3: gelb, PowerGuard:LED3MM
- added POWER1: AC-05-3, PowerGuard:AC-05-3
- added R3: 220, PowerGuard:R_10MM0207/10
- added U$1: WARNLABLE_BLITZ_KLEIN, PowerGuard:WARNLABLE_BLITZ_KLEIN
- added U$2: LOGO_RAUCHSCHWALBE_KLEIN, PowerGuard:LOGO_RAUCHSCHWALBE_KLEIN
- LED1: value red -> rot; device led:LED3MM -> PowerGuard:LED3MM
- LED2: device led:LED3MM -> PowerGuard:LED3MM
- LS_SSR1: value BOB-12009 -> LEVELSHIFTER; device BOB-12009:BOB-12009 -> PowerGuard:LEVELSHIFTER
- R1, R4: device rcl:R-EU_0204/7 -> PowerGuard:R_10MM0207/10
- R2: value 220 -> 330; device rcl:R-EU_0204/7 -> PowerGuard:R_10MM0207/10
- U1: value ESP32-DEVKITC-32D -> ESP32-DEV-KIT-V4; device ESP32-DEVKITC-32D:ESP32-DEVKITC-32D -> PowerGuard:ESP32-DEV-KIT-V4
Connections:
- removed net GND$2: JP1.3, LED1.C, LED2.C, LS_SSR1.GND, U1.GND1, U1.GND2, U1.GND3, X2-3.S, X3-3.S, X4-1.KL
- removed net N$13: U1.IO35
- removed net N$22: U1.SENSOR_VP
- removed net N$3: U1.IO34
- removed net VDD3$13: LS_SSR1.LV, R4.1, U1.3V3, X2-1.S, X3-1.S
- removed net VDD5$3: JP1.4, LS_SSR1.HV, U1.EXT_5V, X4-2.KL
- new net +3V3: CON1.1, CON2.1, LS_SSR1.LV, R4.1, U1.3V3
- new net +5V: CON3.1, JP1.4, LS_SSR1.HV, POWER1.+V, U1.EXT_5V
- new net GND: CON1.3, CON2.3, CON3.2, JP1.3, LED1.C, LED2.C, LED3.C, LS_SSR1.GND, POWER1.-V, U1.GND1, U1.GND2, U1.GND3
- new net N$5: LED3.A, R3.2
- new net N$9: R3.1, U1.IO22
- new net PHASE_L: CON4.1, POWER1.AC/L
- new net PHASE_N: CON4.2, POWER1.AC/N
- net N$11: now also CON1.2, CON2.2; no longer X2-2.S, X3-2.S
Other:
- note added: "L 230V"
- note added: "N 230V"
- note removed: "+12V"
- note removed: "230V"
- moved on the sheet: JP1, LED1, LED2, LS_SSR1, R1, R2, R4, U1
